File: Controller Board.brd (EAGLE design)
At the start: 50 x 37 mm, 31 parts, among them J2 ICSP, J3 Serial, J5 SW1, J6 SW2, Q2 MOSFET-NCHANNEL, U1 ATMEGA328P_TQFP

Commit message: Add files via upload
Parts:
- added C7: 1u, SparkFun-Passives:0603-CAP
- added R7: 1kR, SparkFun-Resistors:0603-RES
- added R8: 10kR, resistor:R0603
- 1: device jameslbr:CRYSTAL-OSC-SMD-5X3.2-2PAD -> jameslbr:CRYSTAL-OSC-SMD-5X3.2
- C1, C2: device resistor:C0805 -> resistor:C0603
- C3, C6: device adafruit:C0805 -> adafruit:C0603
- C4: device SparkFun-Capacitors:CPOL-RADIAL-10UF-25V -> SparkFun-Passives:0603-CAP
- C5: device SparkFun-Capacitors:CPOL-RADIAL-100UF-25V -> SparkFun-Capacitors:PANASONIC_D
- R1, R2, R3, R4, R5, R6: device resistor:M0805 -> resistor:R0603
- moved R5 25.1 mm to (71.0, 44.5), turned to 0 degrees
- moved R1 19.0 mm to (37.1, 23.1), turned to 270 degrees
- moved C6 17.1 mm to (41.4, 28.4)
- moved R2 15.1 mm to (64.5, 47.6), turned to 0 degrees
- moved R4 15.0 mm to (57.5, 47.4), turned to 0 degrees
- moved C1 12.6 mm to (39.5, 25.5), turned to 90 degrees
- moved J3 11.2 mm to (28.9, 34.7)
- moved C2 10.2 mm to (49.0, 26.0)
- moved POWER 10.0 mm to (30.0, 48.0)
- moved C4 9.83 mm to (46.0, 41.5), turned to 90 degrees
- moved R3 9.14 mm to (50.5, 47.3), turned to 0 degrees
- moved S1 7.00 mm to (31.7, 22.2)
- moved J2 6.41 mm to (29.0, 28.0)
- moved C3 4.73 mm to (43.0, 41.5), turned to 90 degrees
- moved 1 1.57 mm to (44.3, 25.0), turned to 180 degrees
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Connections:
- removed net GND-ISO: FAN.2, Q2.3, V+.2
- new net N$10: C7.1, Q2.1, R7.2, R8.1
- net 5V: now also C5.+; no longer C5.1
- net GND: now also C5.-, C7.2, FAN.2, Q2.3, R7.1, V+.2; no longer C5.2
- net N$1: now also 1.3; no longer 1.6
- net N$9: now also R8.2; no longer Q2.1
Routing:
- net N$10: track 0.00 -> 66.1 mm
- net N$9: track 34.2 -> 3.60 mm, vias 1 -> 0
- net N$17: track 32.6 -> 2.60 mm
- net GND-ISO: track 27.1 -> 0.00 mm
- net G: track 54.1 -> 28.3 mm
- net 5V: track 118.6 -> 97.3 mm
- net E: track 32.2 -> 51.6 mm, vias 1 -> 0
- net N$3: track 19.1 -> 2.34 mm
- net N$5: track 19.2 -> 2.50 mm, vias 1 -> 0
- net N$18: track 47.0 -> 30.9 mm, vias 0 -> 1
- net N$2: track 19.0 -> 7.51 mm
- net N$4: track 13.6 -> 2.56 mm
- net RXD: track 22.1 -> 12.2 mm, vias 1 -> 0
- net TXD: track 20.0 -> 11.5 mm, vias 1 -> 0
- net SCK: track 31.7 -> 23.7 mm, vias 2 -> 1
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Other:
- board text removed: "C2"
