File: Controller Board.sch (EAGLE design)
At the start: 31 parts, among them J2 ICSP, J3 Serial, J5 SW1, J6 SW2, Q2 MOSFET-NCHANNEL, U1 ATMEGA328P_TQFP

Commit message: Add files via upload
Parts:
- added C7: 1u, SparkFun-Passives:CAP0603-CAP
- added R7: 1kR, SparkFun-Resistors:RESISTOR0603
- added R8: 10kR, resistor:R-EU_R0603
- 1: device jameslbr:CRYSTAL2 -> jameslbr:CRYSTAL4
- C1, C2: device resistor:C-EUC0805 -> resistor:C-EUC0603
- C3, C6: device adafruit:C-USC0805 -> adafruit:C-USC0603
- C4: device SparkFun-Capacitors:CAP_POLPTH2 -> SparkFun-Passives:CAP0603-CAP
- C5: device SparkFun-Capacitors:CAP_POLPTH1 -> SparkFun-Capacitors:CAP_POLD
- R1, R2, R3, R4, R5, R6: device resistor:R-EU_M0805 -> resistor:R-EU_R0603
Connections:
- removed net GND-ISO: FAN.2, Q2.S, V+.2
- new net N$10: C7.1, Q2.G, R7.2, R8.1
- net 5V: now also C4.1; no longer C4.+
- net GND: now also C4.2, C7.2, FAN.2, Q2.S, R7.1, V+.2; no longer C4.-
- net N$9: now also R8.2; no longer Q2.G
